File: hardware/NixieClock_MainBoard/NixieClock_MainBoard/SENSOR.kicad_sch (KiCad schematic)
At the start: 0 parts

Commit message: layout mainboard
Parts:
- added C7: 100nF, Capacitor_SMD:C_0603_1608Metric, symbol Device:C
- added C8: 1u0, Capacitor_SMD:C_0603_1608Metric, symbol Device:C
Connections:
- new net +3.3V: C7.1, C8.1
- new net GND: C7.2, C8.2
