File: hardware/NixieClock_MainBoard/NixieClock_MainBoard/PWR_USB.kicad_sch (KiCad schematic)
At the start: 9 parts, among them J6 USB_C_Receptacle_USB2.0_16P, Q1 BC847, Q2 BC847, U2 R-78C3.3-1.0, U3 FT230XQ

Commit message: update pcb. distance between fpc-connector corrected
Parts:
- removed U3: FT230XQ, Package_DFN_QFN:QFN-16-1EP_4x4mm_P0.65mm_EP2.1x2.1mm, symbol Interface_USB:FT230XQ
- added U3: FT234XD, Package_DFN_QFN:DFN-12-1EP_3x3mm_P0.45mm_EP1.65x2.38mm, symbol ownSymbols:FT234XD
- J6: footprint Connector_USB:USB_C_Receptacle_G-Switch_GT-USB-7010ASV -> Connector_USB:USB_C_Receptacle_GCT_USB4110
Connections:
- net +3.3V: now also U3.4 (VCC), U3.9 (VCCIO)
- net GND: now also U3.5 (GND)
- net MCU_RXD: now also U3.7 (TXD)
- net MCU_TXD: now also U3.10 (RXD)
- net at J6.A6 (D+), J6.B6 (D+): now also U3.12 (USBDP)
- net at J6.A7 (D-), J6.B7 (D-): now also U3.1 (USBDM)
Changed lines of the file:
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@@
 	(paper "A4")
-	(junction
-		(at 147.32 92.71)
-		(diameter 0)
-		(color 0 0 0 0)
-	)
 	(junction
 		(at 203.2 101.6)
@@
 	)
 	(junction
-		(at 144.78 92.71)
-		(diameter 0)
-		(color 0 0 0 0)
-	)
-	(junction
 		(at 69.85 69.85)
 		(diameter 0)
@@
 	(wire
 		(pts
-			(xy 147.32 90.17) (xy 147.32 92.71)
-		)
-		(stroke
-			(width 0)
-			(type default)
-		)
-	)
-	(wire
-		(pts
 			(xy 224.79 116.84) (xy 224.79 119.38)
 		)
@@
 	(wire
 		(pts
-			(xy 147.32 92.71) (xy 144.78 92.71)
-		)
-		(stroke
-			(width 0)
-			(type default)
-		)
-	)
-	(wire
-		(pts
 			(xy 224.79 101.6) (xy 203.2 101.6)
 		)
@@
 	(wire
 		(pts
-			(xy 144.78 90.17) (xy 144.78 92.71)
+			(xy 144.78 90.17) (xy 144.78 96.52)
 		)
 		(stroke
@@
 	(wire
 		(pts
-			(xy 149.86 92.71) (xy 147.32 92.71)
-		)
-		(stroke
-			(width 0)
-			(type default)
-		)
-	)
-	(wire
-		(pts
-			(xy 149.86 90.17) (xy 149.86 92.71)
-		)
-		(stroke
-			(width 0)
-			(type default)
-		)
-	)
-	(wire
-		(pts
 			(xy 224.79 99.06) (xy 224.79 96.52)
-		)
-		(stroke
-			(width 0)
-			(type default)
-		)
-	)
-	(wire
-		(pts
-			(xy 144.78 92.71) (xy 144.78 96.52)
 		)
 		(stroke
@@
 	)
 	(symbol
+		(lib_id "ownSymbols:FT234XD")
+		(at 147.32 71.12 0)
+		(unit 1)
+		(exclude_from_sim no)
+		(in_bom yes)
+		(on_board yes)
+		(dnp no)
+		(fields_autoplaced yes)
+		(property "Reference" "U3"
+			(at 146.9741 88.9 0)
+			(effects
+				(font
+					(size 1.27 1.27)
+				)
+				(justify left)
+			)
+		)
+		(property "Value" "FT234XD"
+			(at 146.9741 91.44 0)
+			(effects
+				(font
+					(size 1.27 1.27)
+				)
+				(justify left)
+			)
+		)
+		(property "Footprint" "Package_DFN_QFN:DFN-12-1EP_3x3mm_P0.45mm_EP1.65x2.38mm"
+			(at 146.558 72.644 0)
+			(effects
+				(font
+					(size 1.27 1.27)
+				)
+				(hide yes)
+			)
+		)
+		(property "Datasheet" "https://ftdichip.com/wp-content/uploads/2024/05/DS_FT234XD.pdf"
+			(at 146.304 74.676 0)
+			(effects
+				(font
+					(size 1.27 1.27)
+				)
+				(hide yes)
+			)
+		)
+		(property "Description" "USB Full Speed to Basic UART IC with USB Charger Detection, DFN-12"
+			(at 146.558 70.104 0)
+			(effects
+				(font
+					(size 1.27 1.27)
+				)
+				(hide yes)
+			)
+		)
+		(pin "11"
+		)
+		(pin "12"
+		)
+		(pin "5"
+		)
+		(pin "6"
+		)
+		(pin "7"
+		)
+		(pin "8"
+		)
+		(pin "9"
+		)
+		(pin "10"
+		)
+		(pin "3"
+		)
+		(pin "1"
+		)
+		(pin "2"
+		)
+		(pin "4"
+		)
+		(instances
+			(project "NixieClock_MainBoard"
+				(path "/5ddb5910-d1ea-4e23-971a-19156fc3bbe9/951b3c7b-3f91-4669-9ecb-90f69d4a4e63"
+					(reference "U3")
+					(unit 1)
+				)
+			)
+		)
+	)
+	(symbol
 		(lib_id "power:GND")
 		(at 105.41 50.8 0)
@@
 	)
 	(symbol
-		(lib_id "Interface_USB:FT230XQ")
-		(at 147.32 72.39 0)
-		(unit 1)
-		(exclude_from_sim no)
-		(in_bom yes)
-		(on_board yes)
-		(dnp no)
-		(fields_autoplaced yes)
-		(property "Reference" "U3"
-			(at 152.0541 53.34 0)
-			(effects
-				(font
-					(size 1.27 1.27)
-				)
-				(justify left)
-			)
-		)
-		(property "Value" "FT230XQ"
-			(at 152.0541 55.88 0)
-			(effects
-				(font
-					(size 1.27 1.27)
-				)
-				(justify left)
-			)
-		)
-		(property "Footprint" "Package_DFN_QFN:QFN-16-1EP_4x4mm_P0.65mm_EP2.1x2.1mm"
-			(at 181.61 87.63 0)
-			(effects
-				(font
-					(size 1.27 1.27)
-				)
-				(hide yes)
-			)
-		)
-		(property "Datasheet" "https://www.ftdichip.com/Support/Documents/DataSheets/ICs/DS_FT230X.pdf"
-			(at 147.32 72.39 0)
-			(effects
-				(font
-					(size 1.27 1.27)
-				)
-				(hide yes)
-			)
-		)
-		(property "Description" "Full Speed USB to Basic UART, QFN-16"
-			(at 147.32 72.39 0)
-			(effects
-				(font
-					(size 1.27 1.27)
-				)
-				(hide yes)
-			)
-		)
-		(pin "17"
-		)
-		(pin "10"
-		)
-		(pin "15"
-		)
-		(pin "14"
-		)
-		(pin "11"
-		)
-		(pin "12"
-		)
-		(pin "13"
-		)
-		(pin "1"
-		)
-		(pin "4"
-		)
-		(pin "6"
-		)
-		(pin "7"
-		)
-		(pin "5"
-		)
-		(pin "2"
-		)
-		(pin "8"
-		)
-		(pin "16"
-		)
-		(pin "3"
-		)
-		(pin "9"
-		)
-		(instances
-			(project "NixieClock_MainBoard"
-				(path "/5ddb5910-d1ea-4e23-971a-19156fc3bbe9/951b3c7b-3f91-4669-9ecb-90f69d4a4e63"
-					(reference "U3")
-					(unit 1)
-				)
-			)
-		)
-	)
-	(symbol
 		(lib_id "power:GND")
 		(at 73.66 92.71 0)
@@
 			)
 		)
-		(property "Footprint" "Connector_USB:USB_C_Receptacle_G-Switch_GT-USB-7010ASV"
+		(property "Footprint" "Connector_USB:USB_C_Receptacle_GCT_USB4110"
 			(at 54.61 69.85 0)
 			(effects

Commit message: layout mainboard
Changed lines of the file:
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@@
 	(text "Wichtig pinout\nprüfen"
 		(exclude_from_sim no)
-		(at 92.964 36.068 0)
+		(at 106.426 29.464 0)
 		(effects
 			(font

Commit message: update mainboard
Parts:
- removed U3: FT234XD, Package_DFN_QFN:DFN-12-1EP_3x3mm_P0.45mm_EP1.65x2.38mm, symbol ownSymbols:FT234XD
- added C12, C14, C16: 100nF, Capacitor_SMD:C_0603_1608Metric, symbol Device:C
- added C13, C15, C17: 1u0, Capacitor_SMD:C_0603_1608Metric, symbol Device:C
- added R23: 12k, Resistor_SMD:R_0603_1608Metric, symbol Device:R
- added U14: CP2102N-Axx-xQFN24, Package_DFN_QFN:QFN-24-1EP_4x4mm_P0.5mm_EP2.6x2.6mm, symbol Interface_USB:CP2102N-Axx-xQFN24
- added U15: CH340C, Package_SO:SOIC-16_3.9x9.9mm_P1.27mm, symbol Interface_USB:CH340C
Connections:
- net +3.3V: now also C12.1, C13.1, C14.1, C15.1, R23.2, U14.5 (VIO), U14.6 (VDD), U14.7 (VREGIN), U15.16 (VCC), U15.4 (V3)
- net DTR: now also U14.23 (~{DTR}), U15.13 (~{DTR})
- net GND: now also C12.2, C13.2, C14.2, C15.2, C16.2, C17.2, U14.2 (GND), U14.25 (GND), U15.1 (GND)
- net MCU_RXD: now also U14.21 (TXD), U15.2 (TXD)
- net MCU_TXD: now also U14.20 (RXD), U15.3 (RXD)
- net RTS: now also U14.19 (~{RTS}), U15.14 (~{RTS})
- net at J6.A7 (D-), J6.B7 (D-): now also U14.4 (D-), U15.6 (UD-)
- net at J6.A6 (D+), J6.B6 (D+): now also U14.3 (D+), U15.5 (UD+)
- net +5V: now reaches J6.A4 (VBUS), J6.A9 (VBUS), J6.B4 (VBUS), J6.B9 (VBUS), U2.1 (IN)
- net +5V: now also C16.1, C17.1, U14.8 (VBUS)
- new net: R23.1, U14.9 (~{RST})
Other:
- note removed: "Wichtig pinout prüfen"
- moved on the sheet: U2
