File: hardware/NixieClock_MainBoard/NixieClock_MainBoard/uC.kicad_sch (KiCad schematic)
At the start: 9 parts, among them U1 ESP32-WROOM-32E

Commit message: update mainboard
Parts:
- added R22: 10k, Resistor_SMD:R_0603_1608Metric, symbol Device:R
Connections:
- net +3.3V: now also R22.1
- net CS_0: now also U1.29 (IO5); no longer U1.23 (IO15)
- net CS_1: now also U1.27 (IO16); no longer U1.13 (IO14)
- net CS_2: now also U1.24 (IO2); no longer U1.16 (IO13)
- net CS_3: now also U1.16 (IO13); no longer U1.29 (IO5)
- net CS_4: now also U1.13 (IO14), R22.2; no longer U1.27 (IO16)
- net ~{RESET}: now also U1.23 (IO15); no longer U1.24 (IO2)
- net WS28XX: now reaches U1.12 (IO27)
Other:
- moved on the sheet: R10, R11, R12, R9
