File: hardware/NixieClock_MainBoard/PWR_USB.kicad_sch (KiCad schematic)
At the start: 17 parts, among them J6 USB_C_Receptacle_USB2.0_16P, Q1 BC847, Q2 BC847, U14 CP2102N-Axx-xQFN24, U15 CH340C, U2 R-78C3.3-1.0

Commit message: V2.0 release fertig.
Changed lines of the file:
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@@
 	(wire
 		(pts
-			(xy 224.79 83.82) (xy 240.03 83.82)
+			(xy 224.79 83.82) (xy 254 83.82)
 		)
 		(stroke
@@
 	(wire
 		(pts
-			(xy 224.79 119.38) (xy 240.03 119.38)
+			(xy 224.79 119.38) (xy 254 119.38)
 		)
 		(stroke
@@
 	(hierarchical_label "IO0"
 		(shape input)
-		(at 240.03 119.38 0)
+		(at 254 119.38 0)
 		(fields_autoplaced yes)
 		(effects
@@
 	(hierarchical_label "EN"
 		(shape input)
-		(at 240.03 83.82 0)
+		(at 254 83.82 0)
 		(fields_autoplaced yes)
 		(effects
@@
 					(unit 1)
 				)
-			)
-		)
-	)
-	(symbol
-		(lib_id "power:GND")
-		(at 233.68 140.97 0)
-		(unit 1)
-		(exclude_from_sim no)
-		(in_bom yes)
-		(on_board yes)
-		(dnp no)
-		(fields_autoplaced yes)
-		(property "Reference" "#PWR010"
-			(at 233.68 147.32 0)
-			(effects
-				(font
-					(size 1.27 1.27)
-				)
-				(hide yes)
-			)
-		)
-		(property "Value" "GND"
-			(at 233.68 146.05 0)
-			(effects
-				(font
-					(size 1.27 1.27)
-				)
-			)
-		)
-		(property "Footprint" ""
-			(at 233.68 140.97 0)
-			(effects
-				(font
-					(size 1.27 1.27)
-				)
-				(hide yes)
-			)
-		)
-		(property "Datasheet" ""
-			(at 233.68 140.97 0)
-			(effects
-				(font
-					(size 1.27 1.27)
-				)
-				(hide yes)
-			)
-		)
-		(property "Description" "Power symbol creates a global label with name \"GND\" , ground"
-			(at 233.68 140.97 0)
-			(effects
-				(font
-					(size 1.27 1.27)
-				)
-				(hide yes)
-			)
-		)
-		(pin "1"
-		)
-		(instances
-			(project "NixieClock_MainBoard"
-				(path "/5ddb5910-d1ea-4e23-971a-19156fc3bbe9/951b3c7b-3f91-4669-9ecb-90f69d4a4e63"
-					(reference "#PWR010")
-					(unit 1)
-				)

Commit message: Hardware V2.1 add NixieClock_MainBoard/NixieClock_Schematic.pdf
Changed lines of the file:
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@@
 (kicad_sch
-	(version 20231120)
+	(version 20250114)
 	(generator "eeschema")
-	(generator_version "8.0")
+	(generator_version "9.0")
 	(paper "A4")
+	(title_block
+		(date "2026-06-07")
+		(rev "2.1")
+	)
 	(junction
 		(at 139.7 43.18)
@@
 	(label "MCU_RXD"
 		(at 180.34 54.61 0)
-		(fields_autoplaced yes)
 		(effects
 			(font
@@
 	(label "MCU_TXD"
 		(at 180.34 57.15 0)
-		(fields_autoplaced yes)
 		(effects
 			(font
@@
 	(label "DTR"
 		(at 191.77 91.44 0)
-		(fields_autoplaced yes)
 		(effects
 			(font
@@
 	(label "RTS"
 		(at 191.77 111.76 0)
-		(fields_autoplaced yes)
 		(effects
 			(font
@@
 		(shape input)
 		(at 254 119.38 0)
-		(fields_autoplaced yes)
 		(effects
 			(font
@@
 		(shape input)
 		(at 254 83.82 0)
-		(fields_autoplaced yes)
 		(effects
 			(font
@@
 		(shape input)
 		(at 232.41 54.61 0)
-		(fields_autoplaced yes)
 		(effects
 			(font
@@
 		(shape input)
 		(at 232.41 57.15 0)
-		(fields_autoplaced yes)
 		(effects
 			(font
